File: pwm_driver_kicad/pwm_driver_kicad.kicad_sch (KiCad schematic)
At the start: 13 parts, among them J1 Bornera, Q1 IRF540, U1 NE555P

Commit message: add reverse current protection schottky diode
Parts:
- removed B1: BSOURCE, symbol Simulation_SPICE:BSOURCE
- removed C1, C2: 10nF, Capacitor_THT:C_Disc_D4.3mm_W1.9mm_P5.00mm, symbol Device:C
- removed D1, D2: 4148, Diode_THT:D_DO-34_SOD68_P7.62mm_Horizontal, symbol Device:D
- removed D3: LED, symbol Device:LED
- removed R1: 10k, Resistor_THT:R_Axial_DIN0207_L6.3mm_D2.5mm_P7.62mm_Horizontal, symbol Device:R_US
- removed R2: 1k, Resistor_THT:R_Axial_DIN0207_L6.3mm_D2.5mm_P7.62mm_Horizontal, symbol Device:R_US
- removed R3: 330, Resistor_THT:R_Axial_DIN0207_L6.3mm_D2.5mm_P7.62mm_Horizontal, symbol Device:R_US
- added C1, C2: 10nF, symbol Device:C_Small
- added D1, D2: 1N4148, symbol Device:D_Small_Filled
- added D3: 1N5819, symbol Device:D_Schottky_Small_Filled
- added R1: 100k, symbol Device:R_Small_US
- added R2: 1k, symbol Device:R_Small_US
- added RL1: 10, symbol Device:R_Small_US
- added V1: 12, symbol Simulation_SPICE:VDC
Connections:
- net GND: now also J1.1 (Pin_3), C1.1, C2.1, R1.2, V1.2; no longer J1.2 (Pin_2)
- net VCC: now also J1.2 (Pin_2), D3.2 (A), RL1.1, V1.1; no longer J1.3 (Pin_1), U1.4 (R), U1.8 (VCC)
- net at U1.7 (DIS): now also Q1.2 (G), U1.3 (Q), D1.2 (A), D2.1 (K), R1.1, R2.1
- net at RV1.1: now also D2.2 (A)
- net at RV1.2, U1.2 (TR), U1.6 (THR): now also C2.2
- net at RV1.3: now also D1.1 (K)
- net at Q1.1 (D): now also J1.3 (Pin_1), RL1.2; no longer J1.1 (Pin_3)
- net at U1.5 (CV): now also C1.2
- new net: D3.1 (K), R2.2, U1.4 (R), U1.8 (VCC)
Other:
- note added: ".tran 10u 1m uic"
- note removed: ".tran 10u 1m"

Commit message: add potentiometer with switch to toggle output
Parts:
- removed RV1: 50k, Potentiometer_THT:Potentiometer_Alps_RK163_Single_Horizontal, symbol Device:R_Potentiometer_US
- added RVS1: 50k, symbol 1_Resistors:Potentiometer_SW_US_Small
Connections:
- net GND: now also R1.1; no longer R1.2
- net VCC: now also RL1.2; no longer RL1.1
- net at C2.2, U1.2 (TR), U1.6 (THR): now also RVS1.2
- net at D1.1 (K): now also RVS1.3
- net at D1.2 (A), D2.1 (K), R2.1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: now also RVS1.4; no longer Q1.2 (G), R1.1
- net at D2.2 (A): now also RVS1.1
- net OUT-: now reaches J1.3 (Pin_1), Q1.1 (D)
- net OUT-: now also RL1.1; no longer RL1.2
- new net: Q1.2 (G), R1.2, RVS1.5
Other:
- note added: ".tran .1u 2m 1m uic"
- note removed: ".tran 10u 1m uic"
- moved on the sheet: C2, D1, R1, RL1
